File: pcb/motherBoard/kicad-pcb/control_core.kicad_sch (KiCad schematic)
At the start: 13 parts, among them U701 STM32F405RGT6 C15742, Y701 16MHz C13738

Commit message: chore: little 3d models and code fix
Parts:
- removed U701: STM32F405RGT6 C15742, JLCIntegrated:LQFP-64_L10.0-W10.0-P0.50-LS12.0-BL, symbol JLCIntegrated:STM32F405RGT6
- removed Y701: 16MHz C13738, Crystal:Crystal_SMD_3225-4Pin_3.2x2.5mm, symbol Device:Crystal
- added C710: 100nF, Capacitor_SMD:C_0402_1005Metric, symbol Device:C
- added U701: STM32F410RBT6, Package_QFP:LQFP-64_10x10mm_P0.5mm, symbol MCU_ST_STM32F4:STM32F410RBTx
- C701, C702: value 12p C1547 -> 100nF
- C703, C704: value 2.2u 10V -> 100nF; footprint Capacitor_SMD:C_0603_1608Metric -> Capacitor_SMD:C_0402_1005Metric
- C705: value 100n -> 2.2uF; footprint Capacitor_SMD:C_0402_1005Metric -> Capacitor_SMD:C_0603_1608Metric
- C706, C707: value 100n -> 100nF
- C708: value 100n -> 1uF; footprint Capacitor_SMD:C_0402_1005Metric -> Capacitor_SMD:C_0603_1608Metric
- C709: value 4.7u -> 4.7uF
- R701: value 100k -> 10k
Connections:
- net HSE_IN is gone; now on net +3V3: C701.1
- net HSE_OUT is gone; now on net +3V3: C702.1
- net VCAP1 is gone; now on net +3V3: C703.1
- net VCAP2 is gone; now on net +3V3: C704.1
- net +3V3: now also U701.1 (VBAT), U701.13 (VDDA), U701.19 (VDD), U701.32 (VDD), U701.48 (VDD), U701.64 (VDD); no longer C705.1
- net BATTERY_SENSE: now also U701.25 (PC5)
- net BOOT0: now also U701.60 (BOOT0)
- net GND: now also C710.2, U701.12 (VSSA), U701.18 (VSS), U701.31 (VSS), U701.47 (VSS), U701.63 (VSS)
- net LORA1_BUSY: now also U701.22 (PA6)
- net LORA1_DIO1: now also U701.51 (PC10)
- net LORA1_NSS: now also U701.8 (PC0)
- net LORA2_BUSY: now also U701.23 (PA7)
- net LORA2_DIO1: now also U701.52 (PC11)
- net LORA2_NSS: now also U701.9 (PC1)
- net LORA3_BUSY: now also U701.56 (PB4)
- net LORA3_DIO1: now also U701.57 (PB5)
- net LORA3_NSS: now also U701.10 (PC2)
- net LORA_RESET_N: now also U701.28 (PB2)
- net LORA_SPI_MISO: now also U701.45 (PA12)
- net LORA_SPI_MOSI: now also U701.61 (PB8)
- net LORA_SPI_SCK: now also U701.26 (PB0)
- net PI_UART_RX: now also U701.17 (PA3)
- net PI_UART_TX: now also U701.16 (PA2)
- net sensor-scl: now also U701.58 (PB6)
- net sensor-sda: now also U701.59 (PB7)
- net stdc14-rst renamed NRST
- net NRST: now also C710.1, U701.7 (NRST)
- new net: C705.1, U701.30 (VCAP1)
- new net BUZZER_EN: U701.20 (PA4)
- new net CRSF_RX: U701.38 (PC7)
- new net CRSF_TX: U701.37 (PC6)
- new net LED_1: U701.33 (PB12)
- new net LED_2: U701.34 (PB13)
- new net LED_3: U701.35 (PB14)
- new net LED_4: U701.36 (PB15)
- new net LED_STATUS: U701.21 (PA5)
- new net MOTOR_IN1: U701.41 (PA8)
- new net MOTOR_IN2: U701.42 (PA9)
- new net SERVO_DOOR: U701.14 (PA0)
- new net SERVO_ELEVON_L: U701.39 (PC8)
- new net SERVO_ELEVON_R: U701.40 (PC9)
- new net SERVO_WINGS: U701.15 (PA1)
- new net SWCLK: U701.49 (PA14)
- new net SWDIO: U701.46 (PA13)
- new net SWO: U701.55 (PB3)
- no-connect marks 3 -> 15
