File: pcb/motherBoard/kicad-pcb/kicad-pcb.kicad_sch (KiCad schematic)
At the start: 63 parts, among them J1 SG90, J2 SG90, J3 SG90, J4 ELRS, J5 Conn_ST_STDC14, J9 solenoid_valve, Q1 IRLZ44N, Q2 2N7002, U10 AMS1117-3.3, U9 TPS54302, Y1 16MHz

Commit message: chore: little 3d models and code fix
Parts:
- removed C1, C2, C3, C4, C9: 100n, Capacitor_SMD:C_0402_1005Metric, symbol Device:C
- removed C10: 4.7u, Capacitor_SMD:C_0603_1608Metric, symbol Device:C
- removed C11, C12: 12p, Capacitor_SMD:C_0402_1005Metric, symbol Device:C
- removed C22, C23: 22u, Capacitor_SMD:C_0603_1608Metric, symbol Device:C
- removed C5: 10u, Capacitor_SMD:C_0603_1608Metric, symbol Device:C
- removed C6: 10n, Capacitor_SMD:C_0603_1608Metric, symbol Device:C
- removed C7, C8: 1u, Capacitor_SMD:C_0603_1608Metric, symbol Device:C
- removed D2: RED, LED_SMD:LED_0603_1608Metric, symbol Device:LED
- removed D6: 1N4007, Diode_THT:D_DO-41_SOD81_P10.16mm_Horizontal, symbol Diode:1N4007
- removed FB1: 120R, Inductor_SMD:L_0603_1608Metric, symbol Device:FerriteBead
- removed J9: solenoid_valve, TerminalBlock:TerminalBlock_MaiXu_MX126-5.0-02P_1x02_P5.00mm, symbol Connector:Screw_Terminal_01x02
- removed Q1: IRLZ44N, Package_TO_SOT_THT:TO-220-3_Vertical, symbol Transistor_FET:IRLZ44N
- removed R1, R6: 10k, Resistor_SMD:R_0402_1005Metric, symbol Device:R
- removed R13, R14, R15, R16: 5k1, Resistor_SMD:R_0402_1005Metric, symbol Device:R
- removed R17, R18: 22R, Resistor_SMD:R_0402_1005Metric, symbol Device:R
- removed R5: 1k5, Resistor_SMD:R_0402_1005Metric, symbol Device:R
- removed R7: 100R, Resistor_SMD:R_0402_1005Metric, symbol Device:R
- removed U10: AMS1117-3.3, Package_TO_SOT_SMD:SOT-223-3_TabPin2, symbol Regulator_Linear:AMS1117-3.3
- removed Y1: 16MHz, Crystal:Crystal_SMD_3225-4Pin_3.2x2.5mm, symbol Device:Crystal_GND24
- C17: footprint Capacitor_SMD:C_0603_1608Metric -> ㅊ멤챠색_능:ㅊ_0805_2012ㅡㄷㅅ걏; ㅡ (none) -> 치21ㅁ106ㅏ묘ㅜㅜㅜㄸ; ㅣㅊㄴㅊ (none) -> ㅊ15850
- J5: value Conn_ST_STDC14 -> STDC14; footprint Connector_PinHeader_1.27mm:PinHeader_2x07_P1.27mm_Vertical -> JLCIntegrated:Samtec_FTSH-107-01-F-DV-K-P-TR; LCSC (none) -> C5276598; MPN (none) -> FTSH-107-01-F-DV-K-P-TR
- R2: value 100k -> 45.3k
- R3: value 13.5k -> 10k
Connections:
- net PI_UART_RX is gone; now on net PI_UART_TX: J5.14 (VCP_TX)
- net +5V: no longer C15.1, C20.1, C21.1, D1.2 (A), L1.2, R2.1
- net PI_UART_TX: no longer J5.13 (VCP_RX)
- net +12V renamed RAW_BAT
- net +3.3V renamed +3V3
- net +3V3: now also C15.1, C20.1, C21.1, D1.2 (A), L1.2, R2.1
- net stdc14-rst renamed NRST
- net stdc14-swclk renamed SWCLK
- net stdc14-swdio renamed SWDIO
- net stdc14-swo renamed SWO
- new net STLINK_TX_TO_MCU: J5.13 (VCP_RX)
- no-connect marks 13 -> 2
Other:
- sheet Safety_Valve_IO renamed Battery_Deployment_Sense
- removed sheet Integrated_ELRS
- note removed: "DC"
- note removed: "solenoid valve"
